Commit message: add digit sensor

File: envs/urdf/ur5_robotiq_140.urdf (robot description, URDF)
Before this commit: robot ur5_robotiq_140, 20 links, 19 joints
Links:
- added link left_digit, mass 0.02; collision mesh filename=../meshes/digit/digit.STL scale=1 1 1; visual mesh filename=../meshes/digit/digit.STL scale=1 1 1
- added link right_digit, mass 0.02; collision mesh filename=../meshes/digit/digit.STL scale=1 1 1; visual mesh filename=../meshes/digit/digit.STL scale=1 1 1
- link left_inner_finger_pad: mass 1. -> 0.02; geometry collision box size=0.03 0.07 0.0075; visual box size=0.027 0.045 0.0075
- link right_inner_finger_pad: mass 1. -> 0.02; geometry collision box size=0.03 0.07 0.0075; visual box size=0.027 0.045 0.0075
Joints:
- added joint left_digit_adapter_joint: type fixed, parent left_inner_finger_pad, child left_digit, origin xyz=0 0.022 0.01 rpy=-3.141592653589793 1.5707963267948966 -1.5707963267948966, axis 0 0 1
- added joint right_digit_adapter_joint: type fixed, parent right_inner_finger_pad, child right_digit, origin xyz=0 0.022 0.01 rpy=-3.141592653589793 1.5707963267948966 -1.5707963267948966, axis 0 0 1
- joint left_inner_finger_pad_joint: origin xyz=0 0.0457554015893473 -0.0272203446692936 rpy=0 0 0 -> xyz=0 0.0257554015893473 -0.0272203446692936 rpy=0 0 0
- joint right_inner_finger_pad_joint: origin xyz=0 0.0457554015893473 -0.0272203446692936 rpy=0 0 0 -> xyz=0 0.0257554015893473 -0.0272203446692936 rpy=0 0 0

Commit message: finish fixing tactile pointcloud!

File: envs/urdf/ur5_robotiq_140.urdf (robot description, URDF)
Before this commit: robot ur5_robotiq_140, 22 links, 21 joints
Joints:
- joint elbow_joint: limit lower=-3.14159265359 upper=3.14159265359 effort=150.0 velocity=3.15 -> lower=-6.28318530718 upper=6.28318530718 effort=150.0 velocity=3.15
- joint shoulder_lift_joint: limit lower=-3.14159265359 upper=3.14159265359 effort=150.0 velocity=3.15 -> lower=-6.28318530718 upper=6.28318530718 effort=150.0 velocity=3.15
- joint shoulder_pan_joint: limit lower=-3.14159265359 upper=3.14159265359 effort=150.0 velocity=3.15 -> lower=-6.28318530718 upper=6.28318530718 effort=150.0 velocity=3.15
- joint wrist_1_joint: limit lower=-3.14159265359 upper=3.14159265359 effort=28.0 velocity=3.2 -> lower=-6.28318530718 upper=6.28318530718 effort=28.0 velocity=3.2
- joint wrist_2_joint: limit lower=-3.14159265359 upper=3.14159265359 effort=28.0 velocity=3.2 -> lower=-6.28318530718 upper=6.28318530718 effort=28.0 velocity=3.2
- joint wrist_3_joint: limit lower=-3.14159265359 upper=3.14159265359 effort=28.0 velocity=3.2 -> lower=-6.28318530718 upper=6.28318530718 effort=28.0 velocity=3.2
